Commit message: RPLidar added and working

File: tango_sim_ws/src/tango_description/urdf/materials.xacro (robot description, xacro)
@@ -1,6 +1,27 @@
 <?xml version="1.0" ?>
 <robot name="tango" xmlns:xacro="http://www.ros.org/wiki/xacro" >
-<material name="silver">
-  <color rgba="0.700 0.700 0.700 1.000"/>
-</material>
+<material name="black">
+  <color rgba="0.0 0.0 0.0 1.0"/>
+  </material>
+  <material name="blue">
+      <color rgba="0.203125 0.23828125 0.28515625 1.0"/>
+  </material>
+  <material name="green">
+      <color rgba="0.0 0.8 0.0 1.0"/>
+  </material>
+  <material name="grey">
+      <color rgba="0.2 0.2 0.2 1.0"/>
+  </material>
+  <material name="orange">
+      <color rgba="1.0 0.423529411765 0.0392156862745 1.0"/>
+  </material>
+  <material name="brown">
+      <color rgba="0.870588235294 0.811764705882 0.764705882353 1.0"/>
+  </material>
+  <material name="red">
+      <color rgba="0.80078125 0.12890625 0.1328125 1.0"/>
+  </material>
+  <material name="white">
+      <color rgba="1.0 1.0 1.0 1.0"/>
+  </material>
 </robot>

File: tango_sim_ws/src/tango_description/urdf/tango.xacro (robot description, xacro)
@@ -2,6 +2,12 @@
 <robot name="tango" xmlns:xacro="http://www.ros.org/wiki/xacro">
 <xacro:include filename="$(find tango_description)/urdf/materials.xacro" />
+<!-- <xacro:include filename="$(find tango_description)/urdf/macros.xacro" /> -->
 <xacro:include filename="$(find tango_description)/urdf/tango.trans" />
 <xacro:include filename="$(find tango_description)/urdf/tango.gazebo" />
+<macro name="cylinder_inertia" params="mass r l">
+  <inertia  ixx="${mass*(3*r*r+l*l)/12}" ixy = "0" ixz = "0"
+            iyy="${mass*(3*r*r+l*l)/12}" iyz = "0"
+            izz="${mass*(r*r)/2}" />
+</macro>
 <link name="base_link">
   <inertial>
@@ -15,5 +21,5 @@
       <mesh filename="package://tango_description/meshes/base_link.stl" scale="0.001 0.001 0.001"/>
     </geometry>
-    <material name="silver"/>
+    <material name="white"/>
   </visual>
   <collision>
@@ -22,4 +28,24 @@
       <mesh filename="package://tango_description/meshes/base_link.stl" scale="0.001 0.001 0.001"/>
     </geometry>
+  </collision>
+</link>
+<link name="sensor_laser">
+  <inertial>
+      <origin xyz="0 0 0" rpy="0 0 0" />
+      <mass value="1" />
+      <xacro:cylinder_inertia mass="1" r="0.033" l="0.02" />
+  </inertial>
+  <visual>
+      <origin xyz="0 0 0" rpy="0 0 0" />
+      <geometry>
+      <cylinder radius="0.033" length="0.02"/>
+      </geometry>
+      <material name="blue" />
+  </visual>
+  <collision>
+      <origin xyz="0 0 0" rpy="0 0 0"/>
+      <geometry>
+      <cylinder radius="0.033" length="0.02"/>
+      </geometry>
   </collision>
 </link>
@@ -35,5 +61,5 @@
       <mesh filename="package://tango_description/meshes/wheel_right_1.stl" scale="0.001 0.001 0.001"/>
     </geometry>
-    <material name="silver"/>
+    <material name="black"/>
   </visual>
   <collision>
@@ -55,5 +81,5 @@
       <mesh filename="package://tango_description/meshes/wheel_left_1.stl" scale="0.001 0.001 0.001"/>
     </geometry>
-    <material name="silver"/>
+    <material name="black"/>
   </visual>
   <collision>
@@ -64,4 +90,9 @@
   </collision>
 </link>
+<joint name="joint_sensor_laser" type="fixed">
+    <origin xyz="-0.153 -0.150 0.210" rpy="0 0 0"/>
+    <parent link="base_link"/>
+    <child link="sensor_laser"/>
+</joint>
 <joint name="right_rev" type="continuous">
   <origin rpy="0 0 0" xyz="-0.320255 -0.152026 0.056187"/>

Commit message: fixed model joint misalignment

File: tango_sim_ws/src/tango_description/urdf/materials.xacro (robot description, xacro)
@@ -1,5 +1,8 @@
 <?xml version="1.0" ?>
 <robot name="tango" xmlns:xacro="http://www.ros.org/wiki/xacro" >
-<material name="black">
+  <material name="silver">
+    <color rgba="0.700 0.700 0.700 1.000"/>
+  </material>
+  <material name="black">
   <color rgba="0.0 0.0 0.0 1.0"/>
   </material>

File: tango_sim_ws/src/tango_description/urdf/tango.xacro (robot description, xacro)
@@ -11,7 +11,7 @@
 <link name="base_link">
   <inertial>
-    <origin rpy="0 0 0" xyz="-0.16178693932823193 -0.1338655452414066 0.11034012029652868"/>
-    <mass value="1.222219902266934"/>
-    <inertia ixx="0.012663" ixy="0.00086" ixz="0.000171" iyy="0.010559" iyz="-0.000482" izz="0.018404"/>
+    <origin rpy="0 0 0" xyz="0.00016953576698395381 -0.003784058871619607 0.04856680225483841"/>
+    <mass value="0.9483275242628453"/>
+    <inertia ixx="0.010174" ixy="-0.000103" ixz="-4.4e-05" iyy="0.009278" iyz="0.000222" izz="0.015459"/>
   </inertial>
   <visual>
@@ -20,5 +20,5 @@
       <mesh filename="package://tango_description/meshes/base_link.stl" scale="0.001 0.001 0.001"/>
     </geometry>
-    <material name="white"/>
+    <material name="silver"/>
   </visual>
   <collision>
@@ -49,19 +49,39 @@
   </collision>
 </link>
+<link name="wheel_left_1">
+  <inertial>
+    <origin rpy="0 0 0" xyz="-0.16628589477289957 5.602462880330887e-14 -7.487718159456705e-16"/>
+    <mass value="0.5462470782161397"/>
+    <inertia ixx="0.001184" ixy="-0.0" ixz="0.0" iyy="0.000606" iyz="-0.0" izz="0.000606"/>
+  </inertial>
+  <visual>
+    <origin rpy="0 0 0" xyz="-0.0 -0.0 0.0"/>
+    <geometry>
+      <mesh filename="package://tango_description/meshes/wheel_left_1.stl" scale="0.001 0.001 0.001"/>
+    </geometry>
+    <material name="silver"/>
+  </visual>
+  <collision>
+    <origin rpy="0 0 0" xyz="-0.0 -0.0 0.0"/>
+    <geometry>
+      <mesh filename="package://tango_description/meshes/wheel_left_1.stl" scale="0.001 0.001 0.001"/>
+    </geometry>
+  </collision>
+</link>
 <link name="wheel_right_1">
   <inertial>
-    <origin rpy="0 0 0" xyz="-0.001378146385077439 -3.803152259784781e-08 2.701640913968517e-07"/>
-    <mass value="0.5465183547417778"/>
-    <inertia ixx="0.001184" ixy="-0.0" ixz="-0.0" iyy="0.000606" iyz="-0.0" izz="0.000606"/>
+    <origin rpy="0 0 0" xyz="0.16473964498315097 1.3460578998617458e-14 5.271833050320694e-16"/>
+    <mass value="0.546247078216141"/>
+    <inertia ixx="0.001184" ixy="-0.0" ixz="0.0" iyy="0.000606" iyz="-0.0" izz="0.000606"/>
   </inertial>
   <visual>
-    <origin rpy="0 0 0" xyz="0.320255 0.152026 -0.056187"/>
+    <origin rpy="0 0 0" xyz="-0.0 -0.0 0.0"/>
     <geometry>
       <mesh filename="package://tango_description/meshes/wheel_right_1.stl" scale="0.001 0.001 0.001"/>
     </geometry>
-    <material name="black"/>
+    <material name="silver"/>
   </visual>
   <collision>
-    <origin rpy="0 0 0" xyz="0.320255 0.152026 -0.056187"/>
+    <origin rpy="0 0 0" xyz="-0.0 -0.0 0.0"/>
     <geometry>
       <mesh filename="package://tango_description/meshes/wheel_right_1.stl" scale="0.001 0.001 0.001"/>
@@ -69,44 +89,20 @@
   </collision>
 </link>
-<link name="wheel_left_1">
-  <inertial>
-    <origin rpy="0 0 0" xyz="0.0013779841244327354 -3.8031565174900805e-08 2.7018644199044983e-07"/>
-    <mass value="0.5465183547417778"/>
-    <inertia ixx="0.001184" ixy="-0.0" ixz="-0.0" iyy="0.000606" iyz="0.0" izz="0.000606"/>
-  </inertial>
-  <visual>
-    <origin rpy="0 0 0" xyz="-0.013525 0.152026 -0.056387"/>
-    <geometry>
-      <mesh filename="package://tango_description/meshes/wheel_left_1.stl" scale="0.001 0.001 0.001"/>
-    </geometry>
-    <material name="black"/>
-  </visual>
-  <collision>
-    <origin rpy="0 0 0" xyz="-0.013525 0.152026 -0.056387"/>
-    <geometry>
-      <mesh filename="package://tango_description/meshes/wheel_left_1.stl" scale="0.001 0.001 0.001"/>
-    </geometry>
-  </collision>
-</link>
 <joint name="joint_sensor_laser" type="fixed">
-    <origin xyz="-0.153 -0.150 0.210" rpy="0 0 0"/>
+    <origin xyz="0.0 0.0 0.1496" rpy="0 0 0"/>
     <parent link="base_link"/>
     <child link="sensor_laser"/>
 </joint>
-<joint name="right_rev" type="continuous">
-  <origin rpy="0 0 0" xyz="-0.320255 -0.152026 0.056187"/>
+<joint name="Rev15" type="continuous">
+  <origin rpy="0 0 0" xyz="0.0 0.0 0.0"/>
+  <parent link="base_link"/>
+  <child link="wheel_left_1"/>
+  <axis xyz="-1.0 0.0 -0.0"/>
+</joint>
+<joint name="Rev16" type="continuous">
+  <origin rpy="0 0 0" xyz="0.0 0.0 0.0"/>
   <parent link="base_link"/>
   <child link="wheel_right_1"/>
-  <axis xyz="1.0 0.0 0.0"/>
-  <limit effort="100" velocity="100"/>
-  <joint_properties damping="0.0" friction="0.0"/>
-</joint>
-<joint name="left_rev" type="continuous">
-  <origin rpy="0 0 0" xyz="0.013525 -0.152026 0.056387"/>
-  <parent link="base_link"/>
-  <child link="wheel_left_1"/>
-  <axis xyz="1.0 -0.0 -0.0"/>
-  <limit effort="100" velocity="100"/>
-  <joint_properties damping="0.0" friction="0.0"/>
+  <axis xyz="-1.0 -0.0 0.0"/>
 </joint>
 </robot>
