Commit message: Diff_drive plugin added and tested.

File: tango_sim_ws/src/tango_description/urdf/tango.xacro (robot description, xacro)
@@ -98,5 +98,7 @@
   <parent link="base_link"/>
   <child link="wheel_right_1"/>
-  <axis xyz="-1.0 0.0 0.0"/>
+  <axis xyz="1.0 0.0 0.0"/>
+  <limit effort="100" velocity="100"/>
+  <joint_properties damping="0.0" friction="0.0"/>
 </joint>
 <joint name="left_rev" type="continuous">
@@ -105,4 +107,6 @@
   <child link="wheel_left_1"/>
   <axis xyz="1.0 -0.0 -0.0"/>
+  <limit effort="100" velocity="100"/>
+  <joint_properties damping="0.0" friction="0.0"/>
 </joint>
 </robot>

Commit message: added xacro: tag for noetic

File: tango_sim_ws/src/tango_description/urdf/tango.xacro (robot description, xacro)
@@ -4,9 +4,9 @@
 <xacro:include filename="$(find tango_description)/urdf/tango.trans" />
 <xacro:include filename="$(find tango_description)/urdf/tango.gazebo" />
-<macro name="cylinder_inertia" params="mass r l">
+<xacro:macro name="cylinder_inertia" params="mass r l">
   <inertia  ixx="${mass*(3*r*r+l*l)/12}" ixy = "0" ixz = "0"
             iyy="${mass*(3*r*r+l*l)/12}" iyz = "0"
             izz="${mass*(r*r)/2}" />
-</macro>
+</xacro:macro>
 <link name="base_link">
   <inertial>

Commit message: dummy link and physics engine step size

File: tango_sim_ws/src/tango_description/urdf/tango.xacro (robot description, xacro)
@@ -9,4 +9,5 @@
             izz="${mass*(r*r)/2}" />
 </xacro:macro>
+<link name="dummy_link" />
 <link name="base_link">
   <inertial>
@@ -89,4 +90,8 @@
   </collision>
 </link>
+<joint name="dummy_joint" type="fixed">
+<parent link="dummy_link"/>
+<child link="base_link"/>
+</joint>
 <joint name="joint_sensor_laser" type="fixed">
     <origin xyz="0.0 0.0 0.1496" rpy="0 0 0"/>

File: tango_sim_ws/src/tango_description/urdf/tango.xacro.urdf (robot description, URDF)
Before this commit: robot tango, 4 links, 3 joints
Links:
- added link dummy_link
Joints:
- added joint dummy_joint: type fixed, parent dummy_link, child base_link

Commit message: obs.py fixed, lidar pose fixed

File: tango_sim_ws/src/tango_description/urdf/tango.xacro (robot description, xacro)
@@ -95,5 +95,5 @@
 </joint>
 <joint name="joint_sensor_laser" type="fixed">
-    <origin xyz="0.0 0.0 0.1496" rpy="0 0 0"/>
+    <origin xyz="0.0 0.0 0.1496" rpy="0 0 1.570796"/>
     <parent link="base_link"/>
     <child link="sensor_laser"/>
